Commit message: Challenge 2 - URDF and Launcher Created

File: Week2/puzzlebot_urdf_ROS/urdf/puzzlebot.urdf (robot description, URDF)
Before this commit: robot Puzzlebot_Jetson_Lidar_Ed., 0 links, 0 joints
Links:
- added link base_footprint
- added link base_link, mass 1.0; collision box size=0.19 0.15 0.10; visual mesh filename=package://puzzlebot_urdf_ROS/meshes/Puzzlebot_Jetson_Lidar_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 scale=1 1 1
- added link caster, mass 0.05; collision sphere radius=0.015; visual mesh filename=package://puzzlebot_urdf_ROS/meshes/Puzzlebot_Caster_Wheel.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 scale=1 1 1
- added link odom
- added link wheel_l, mass 0.1; collision cylinder length=0.02 radius=0.05; visual mesh filename=package://puzzlebot_urdf_ROS/meshes/Puzzlebot_Wheel.stl scale=1 1 1
- added link wheel_r, mass 0.1; collision cylinder length=0.02 radius=0.05; visual mesh filename=package://puzzlebot_urdf_ROS/meshes/Puzzlebot_Wheel.stl scale=1 1 1
Joints:
- added joint base_footprint_to_base_link: type fixed, parent base_footprint, child base_link, origin xyz=0.0 0.0 0.06 rpy=0.0 0.0 0.0
- added joint base_link_to_caster: type fixed, parent base_link, child caster, origin xyz=0.0 -0.075 -0.055 rpy=0.0 0.0 0.0
- added joint base_link_to_wheel_l: type continuous, parent base_link, child wheel_l, origin xyz=-0.084 0.053 -0.01 rpy=0 1.5708 0.0, axis 0 0 1
- added joint base_link_to_wheel_r: type continuous, parent base_link, child wheel_r, origin xyz=0.084 0.053 -0.01 rpy= 3.1416  1.5708 0.0, axis 0 0 1
- added joint odom_to_base_footprint: type fixed, parent odom, child base_footprint, origin xyz=0.0 0.0 0.0 rpy=0.0 0.0 0.0

Commit message: FIXED movement of base footprint and added odometry to the robot in open loop

File: Week2/puzzlebot_urdf_ROS/urdf/puzzlebot.urdf (robot description, URDF)
Before this commit: robot puzzlebot, 6 links, 5 joints
Links:
- removed link odom
- link base_link: mass 1.0 -> None; geometry visual mesh filename=package://puzzlebot_urdf_ROS/meshes/Puzzlebot_Jetson_Lidar_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 scale=1 1 1
- link caster: mass 0.05 -> None; geometry visual mesh filename=package://puzzlebot_urdf_ROS/meshes/Puzzlebot_Caster_Wheel.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 scale=1 1 1
- link wheel_l: mass 0.1 -> None; geometry visual mesh filename=package://puzzlebot_urdf_ROS/meshes/Puzzlebot_Wheel.stl scale=1 1 1
- link wheel_r: mass 0.1 -> None; geometry visual mesh filename=package://puzzlebot_urdf_ROS/meshes/Puzzlebot_Wheel.stl scale=1 1 1
Joints:
- removed joint odom_to_base_footprint
- joint base_link_to_wheel_l: origin xyz=-0.084 0.053 -0.01 rpy=0 1.5708 0.0 -> xyz=-0.084 0.053 -0.01 rpy=3.1416 -1.5708 0.0
- joint base_link_to_wheel_r: origin xyz=0.084 0.053 -0.01 rpy= 3.1416  1.5708 0.0 -> xyz=0.084 0.053 -0.01 rpy=0.0 -1.5708 0.0

Commit message: Fixed duplicate inversions of Wheel_l

File: Week2/puzzlebot_urdf_ROS/urdf/puzzlebot.urdf (robot description, URDF)
Before this commit: robot puzzlebot, 5 links, 4 joints
Joints:
- joint base_link_to_wheel_l: origin xyz=-0.084 0.053 -0.01 rpy=3.1416 -1.5708 0.0 -> xyz=-0.084 0.053 -0.01 rpy=0.0 -1.5708 0.0
