Commit message: URDF

File: Week3/puzzlebot_sim3/urdf/puzzlebot.urdf (robot description, URDF)
Before this commit: robot Puzzlebot_Jetson_Lidar_Ed., 7 links, 6 joints
Links:
- removed link camera_base_link
- removed link caster_holder_link
- removed link lidar_base_link
- removed link wheel_left_link
- removed link wheel_right_link
- added link caster; visual mesh filename=package://puzzlebot_urdf_ROS/meshes/Puzzlebot_Caster_Wheel.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 scale=1 1 1
- added link wheel_l; visual mesh filename=package://puzzlebot_urdf_ROS/meshes/Puzzlebot_Wheel.stl scale=1 1 1
- added link wheel_r; visual mesh filename=package://puzzlebot_urdf_ROS/meshes/Puzzlebot_Wheel.stl scale=1 1 1
- link base_link: geometry visual mesh filename=package://puzzlebot_urdf_ROS/meshes/Puzzlebot_Jetson_Lidar_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 scale=1 1 1
Joints:
- removed joint base_link_joint
- removed joint camera_base_joint
- removed joint caster_holder_joint
- removed joint lidar_base_joint
- removed joint wheel_left_joint
- removed joint wheel_right_joint
- added joint base_footprint_to_base_link: type fixed, parent base_footprint, child base_link, origin xyz=0.0 0.0 0.06 rpy=0.0 0.0 0.0
- added joint base_link_to_caster: type fixed, parent base_link, child caster, origin xyz=0.0 -0.075 -0.055 rpy=0.0 0.0 0.0
- added joint base_link_to_wheel_l: type continuous, parent base_link, child wheel_l, origin xyz=-0.084 0.053 -0.01 rpy=0.0 -1.5708 0.0, axis 0 0 1
- added joint base_link_to_wheel_r: type continuous, parent base_link, child wheel_r, origin xyz=0.084 0.053 -0.01 rpy=0.0 -1.5708 0.0, axis 0 0 1

Commit message: Fixed URDF, Changes in Localization so heading of Odom Correct

File: Week3/puzzlebot_sim3/urdf/puzzlebot.urdf (robot description, URDF)
Before this commit: robot puzzlebot, 5 links, 4 joints
Joints:
- joint base_footprint_to_base_link: origin xyz=0.0 0.0 0.06 rpy=0.0 0.0 0.0 -> xyz=0.0 0.0 0.06 rpy=0.0 0.0 -1.5708
- joint base_link_to_wheel_l: origin xyz=-0.084 0.053 -0.01 rpy=0.0 -1.5708 0.0 -> xyz=-0.084 0.054 -0.01 rpy=0.0 -1.5708 0.0
- joint base_link_to_wheel_r: origin xyz=0.084 0.053 -0.01 rpy=0.0 -1.5708 0.0 -> xyz=0.084 0.054 -0.01 rpy=0.0 -1.5708 0.0
