Commit message: Color update

File: Week7/puzzlebot_gazebo_sim/puzzlebot_description/urdf/mcr2_mechanical/puzzlebot_hacker_base.urdf.xacro (robot description, xacro)
@@ -11,5 +11,5 @@
                 <mesh filename="file://${mesh_puzzlebot_chassis}"/>
             </geometry>
-            <material name="yellow"/>
+            <material name="green"/>
         </visual>
         <collision>

File: Week7/puzzlebot_gazebo_sim/puzzlebot_description/urdf/mcr2_mechanical/puzzlebot_jetson_base.urdf.xacro (robot description, xacro)
@@ -11,5 +11,5 @@
                 <mesh filename="file://${mesh_puzzlebot_chassis}"/>
             </geometry>
-            <material name="yellow"/>
+            <material name="green"/>
         </visual>
         <collision>

File: Week7/puzzlebot_gazebo_sim/puzzlebot_description/urdf/mcr2_mechanical/puzzlebot_jetson_lidar_base.urdf.xacro (robot description, xacro)
@@ -11,5 +11,5 @@
                 <mesh filename="file://${mesh_puzzlebot_chassis}"/>
             </geometry>
-            <material name="yellow"/>
+            <material name="green"/>
         </visual>
         <collision>
